File: kicad/power-control_2.kicad_pcb (KiCad board)
At the start: 2 copper layers, 92 x 60 mm, 37 parts, among them J1 PSU_POWER, J10 USB_4_SOCKET, J3 PINHD_2x5_Male, J4 Conn_01x08_Pin, J5 USB_A, J6 USB_A, J7 USB_3_SOCKET, J9 Conn_01x04_Pin, SW1 Push_Button, SW2 Push_Button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

Commit message: full update
Parts:
- removed the C10 at (212.8, 85.1)
- removed C12: 100uF_0603, PCM_Capacitor_SMD_AKL:C_0603_1608Metric
- removed the C9 at (190.4, 98.8)
- removed the J1 at (188.4, 72.6)
- removed R14, R15, R17: R_100kOm, PCM_Resistor_SMD_AKL:R_0805_2012Metric
- removed R16: R_47kOm, PCM_Resistor_SMD_AKL:R_0805_2012Metric
- removed R2: 1kOm, PCM_Resistor_THT_AKL_Double:R_Axial_DIN0207_L6.3mm_D2.5mm_P7.62mm_Horizontal
- removed R3, R4: 10kOm, PCM_Resistor_THT_AKL_Double:R_Axial_DIN0207_L6.3mm_D2.5mm_P7.62mm_Horizontal
- added C2: 100uF_16V, PCM_Capacitor_THT_AKL:C_Radial_D5.0mm_H11.0mm_P2.00mm, B.Cu at (107.0, 65.8)
- added C4: 100uF_16V, PCM_Capacitor_THT_AKL:C_Radial_D5.0mm_H11.0mm_P2.00mm, B.Cu at (163.8, 68.0)
- added R10: R_1kOm, PCM_Resistor_SMD_AKL:R_1206_3216Metric, F.Cu at (134.2, 100.8)
- added R11: R_1kOm, PCM_Resistor_SMD_AKL:R_1206_3216Metric, F.Cu at (143.2, 75.1)
- added R12: R_10kOm, PCM_Resistor_SMD_AKL:R_1206_3216Metric, F.Cu at (155.5, 102.5)
- added R5: R_100kOm, PCM_Resistor_SMD_AKL:R_1206_3216Metric, F.Cu at (177.0, 112.9)
- added R6: R_47kOm, PCM_Resistor_SMD_AKL:R_1206_3216Metric, F.Cu at (174.0, 112.9)
- added R7: R_100kOm, PCM_Resistor_SMD_AKL:R_1206_3216Metric, F.Cu at (163.8, 112.6)
- added R8: R_100kOm, PCM_Resistor_SMD_AKL:R_1206_3216Metric, F.Cu at (171.0, 112.9)
- BC1: renamed from power-transistor1; value BC548 -> Q1
- BC2: renamed from reset-transistor1; value BC548 -> Q2
- C10: renamed from C15; footprint PCM_Capacitor_SMD_AKL:C_0603_1608Metric -> PCM_Capacitor_SMD_AKL:C_1206_3216Metric
- C3, C5: value 100uF_0603 -> 100uF_16V; footprint PCM_Capacitor_SMD_AKL:C_0603_1608Metric -> PCM_Capacitor_THT_AKL:C_Radial_D5.0mm_H11.0mm_P2.00mm; moved to B.Cu
- C6: value 100uF_0603 -> 10uF_0603; footprint PCM_Capacitor_SMD_AKL:C_0603_1608Metric -> PCM_Capacitor_SMD_AKL:C_1206_3216Metric
- C7: renamed from C17; footprint PCM_Capacitor_SMD_AKL:C_0603_1608Metric -> PCM_Capacitor_SMD_AKL:C_1206_3216Metric
- C8: renamed from C16; footprint PCM_Capacitor_SMD_AKL:C_0603_1608Metric -> PCM_Capacitor_SMD_AKL:C_1206_3216Metric
- C9: renamed from C13; footprint PCM_Capacitor_SMD_AKL:C_0603_1608Metric -> PCM_Capacitor_SMD_AKL:C_1206_3216Metric
- J1: renamed from J9; moved to B.Cu
- J2: renamed from J6; value USB_A -> USB_1
- J3: renamed from J10; moved to B.Cu
- J5: value USB_A -> USB_2
- J6: renamed from J7; moved to B.Cu
- R1: value 1kOm -> 2.7kOm; footprint PCM_Resistor_THT_AKL_Double:R_Axial_DIN0207_L6.3mm_D2.5mm_P7.62mm_Horizontal -> PCM_Resistor_SMD_AKL:R_1206_3216Metric; moved to F.Cu
- R13: value 2.7kOm -> R_10kOm; footprint PCM_Resistor_THT_AKL_Double:R_Axial_DIN0207_L6.3mm_D2.5mm_P7.62mm_Horizontal -> PCM_Resistor_SMD_AKL:R_1206_3216Metric; moved to F.Cu
- moved J3 110.6 mm to (109.8, 70.3), turned to 180 degrees
- moved C10 61.4 mm to (183.0, 103.2), turned to 0 degrees
- moved J6 60.2 mm to (116.7, 112.1), turned to 180 degrees
- moved CRYSTAL1 52.4 mm to (174.9, 91.2), turned to -90 degrees
- moved C3 51.1 mm to (110.5, 106.2), turned to 180 degrees
- moved C7 48.0 mm to (180.0, 112.9), turned to -90 degrees
- moved C8 47.5 mm to (183.2, 112.9), turned to 90 degrees
- moved C9 47.0 mm to (183.0, 106.5)
- moved C5 44.6 mm to (168.2, 74.2), turned to 180 degrees
- moved U2 39.8 mm to (167.3, 104.3), turned to -90 degrees
- moved C6 23.7 mm to (188.9, 74.2)
- moved R1 23.5 mm to (158.5, 112.5), turned to -90 degrees
- moved R13 22.8 mm to (140.9, 102.6), turned to -90 degrees
- moved BC1 7.96 mm to (136.5, 105.9), turned to 180 degrees
- moved SW3 7.91 mm to (114.3, 68.4), turned to 0 degrees
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- renumbered CRYSTAL2 to CRYSTAL1, J3 to J7, U3 to U2
Connections:
- BC1 pad 2: Net-(R1--) -> Net-(BC1-B)
- C3 pad 1: GND -> /VCC_2
- C3 pad 2: /VCC_2 -> GND
- C5 pad 1: GND -> /VCC_2
- C5 pad 2: /VCC_2 -> GND
- C6 pad 2: /VCC_1 -> /VCC_2
- R1 pad 1: /GPIO9 -> Net-(U2-REXT)
- R1 pad 2: Net-(R1--) -> GND
- R13 pad 1: Net-(U3-REXT) -> /GPIO5
- R13 pad 2: GND -> /GND_ESP
- SW3 pad 2: /GPIO4 -> /GPIO3
- U1 pad 7: unconnected-(U1-GPIO7-Pad7) -> /GPIO7
- U1 pad 9: /GPIO9 -> unconnected-(U1-GPIO9-Pad9)
- U2 pad 10: /DATA_2- -> /DATA_3_SOCKET-
- U2 pad 11: /DATA_2+ -> /DATA_3_SOCKET+
- U2 pad 14: Net-(U3-REXT) -> Net-(U2-REXT)
- U2 pad 4: /DATA_4_SOCKET- -> /ESP_USB_DATA-
- U2 pad 5: /DATA_4_SOCKET+ -> /ESP_USB_DATA+
- U2 pad 6: /DATA_3_SOCKET- -> /DATA_2-
- U2 pad 7: /DATA_3_SOCKET+ -> /DATA_2+
- U2 pad 8: /ESP_USB_DATA- -> /DATA_4_SOCKET-
- U2 pad 9: /ESP_USB_DATA+ -> /DATA_4_SOCKET+
Routing:
- net /VCC_2: track 29.6 -> 355.8 mm, vias 0 -> 11
- net GND: track 295.8 -> 46.7 mm
- net /GND_ESP: track 163.7 -> 26.9 mm, vias 0 -> 2
- net /DATA_4_SOCKET-: track 25.3 -> 77.9 mm, vias 0 -> 2
- net /DATA_4_SOCKET+: track 25.0 -> 76.4 mm, vias 0 -> 2
- net /DATA_3_SOCKET+: track 25.1 -> 69.4 mm
- net /DATA_3_SOCKET-: track 25.1 -> 66.9 mm
- net /GPIO3: track 4.60 -> 44.8 mm, vias 0 -> 2
- net /DATA_U-: track 28.6 -> 64.4 mm
- net /GPIO4: track 43.4 -> 8.41 mm
- net /FP_PW_L+: track 92.7 -> 58.3 mm
- net /FP_PW_L-: track 80.6 -> 51.5 mm
- net /FP_PW_B+: track 44.0 -> 71.8 mm, vias 0 -> 2
- net /VD_3.3: track 0.00 -> 23.7 mm, vias 0 -> 2
- net /DATA_U+: track 43.2 -> 66.5 mm
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- added copper zone on F.Cu, net /GND_ESP
- added copper zone on F.Cu, net GND
Other:
- board size 92 x 60 mm -> 91 x 62 mm
