File: kicad/power-control_2.kicad_sch (KiCad schematic)
At the start: 37 parts, among them J1 Conn_01x02_Pin, J10 USB_4_SOCKET, J3 PINHD_2x5_Male, J4 Conn_01x08_Pin, J5 USB_A, J6 USB_A, J7 USB_3_SOCKET, J9 Conn_01x04_Pin, SW1 Push_Button, SW2 Push_Button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

Commit message: full update
Parts:
- removed C10, C12, C3, C5, C6: 100uF_0603, PCM_Capacitor_SMD_AKL:C_0603_1608Metric, symbol PCM_Capacitor_AKL:C_0603
- removed R1, R2: 1kOm, PCM_Resistor_THT_AKL_Double:R_Axial_DIN0207_L6.3mm_D2.5mm_P7.62mm_Horizontal, symbol PCM_Elektuur:R
- removed R13: 2.7kOm, PCM_Resistor_THT_AKL_Double:R_Axial_DIN0207_L6.3mm_D2.5mm_P7.62mm_Horizontal, symbol PCM_SL_Resistors:Resistor
- removed R14, R15, R17: R_100kOm, PCM_Resistor_SMD_AKL:R_0805_2012Metric, symbol PCM_Resistor_AKL:R_0805
- removed R16: R_47kOm, PCM_Resistor_SMD_AKL:R_0805_2012Metric, symbol PCM_Resistor_AKL:R_0805
- removed R3, R4: 10kOm, PCM_Resistor_THT_AKL_Double:R_Axial_DIN0207_L6.3mm_D2.5mm_P7.62mm_Horizontal, symbol PCM_Elektuur:R
- added C2, C3, C4, C5: 100uF_16V, PCM_Capacitor_THT_AKL:C_Radial_D5.0mm_H11.0mm_P2.00mm, symbol PCM_SL_Capacitors:100uF_16V
- added R1: 2.7kOm, PCM_Resistor_SMD_AKL:R_1206_3216Metric, symbol PCM_Resistor_AKL:R_0603
- added R10, R11: R_1kOm, PCM_Resistor_SMD_AKL:R_1206_3216Metric, symbol PCM_Resistor_AKL:R_1206
- added R12, R13: R_10kOm, PCM_Resistor_SMD_AKL:R_1206_3216Metric, symbol PCM_Resistor_AKL:R_1206
- added R5, R7, R8: R_100kOm, PCM_Resistor_SMD_AKL:R_1206_3216Metric, symbol PCM_Resistor_AKL:R_1206
- added R6: R_47kOm, PCM_Resistor_SMD_AKL:R_1206_3216Metric, symbol PCM_Resistor_AKL:R_1206
- BC1: renamed from power-transistor1; value BC548 -> Q1
- BC2: renamed from reset-transistor1; value BC548 -> Q2
- C10: renamed from C15; footprint PCM_Capacitor_SMD_AKL:C_0603_1608Metric -> PCM_Capacitor_SMD_AKL:C_1206_3216Metric
- C6: renamed from C9; footprint PCM_Capacitor_SMD_AKL:C_0603_1608Metric -> PCM_Capacitor_SMD_AKL:C_1206_3216Metric
- C7: renamed from C17; footprint PCM_Capacitor_SMD_AKL:C_0603_1608Metric -> PCM_Capacitor_SMD_AKL:C_1206_3216Metric
- C8: renamed from C16; footprint PCM_Capacitor_SMD_AKL:C_0603_1608Metric -> PCM_Capacitor_SMD_AKL:C_1206_3216Metric
- C9: renamed from C13; footprint PCM_Capacitor_SMD_AKL:C_0603_1608Metric -> PCM_Capacitor_SMD_AKL:C_1206_3216Metric
- J2: renamed from J6; value USB_A -> USB_1
- J5: value USB_A -> USB_2
- J8: renamed from J1; footprint (none) -> ${KICAD9_3DMODEL_DIR}/Connector_JST.3dshapes/JST_XH_B2B-XH-A_1x02_P2.50mm_Vertical.wrl
- renumbered CRYSTAL2 to CRYSTAL1, J9 to J1, J10 to J3, J7 to J6, J3 to J7, U3 to U2
Connections:
- net DATA_2+: now also U2.7 (DP3); no longer U2.11 (DP1)
- net DATA_2-: now also U2.6 (DM3); no longer U2.10 (DM1)
- net DATA_3_SOCKET+: now also U2.11 (DP1); no longer U2.7 (DP3)
- net DATA_3_SOCKET-: now also U2.10 (DM1); no longer U2.6 (DM3)
- net DATA_4_SOCKET+: now also U2.9 (DP2); no longer U2.5 (DP4)
- net DATA_4_SOCKET-: now also U2.8 (DM2); no longer U2.4 (DM4)
- net ESP_USB_DATA+: now also U2.5 (DP4); no longer U2.9 (DP2)
- net ESP_USB_DATA-: now also U2.4 (DM4); no longer U2.8 (DM2)
- net FP_PW_L+: now also R12.1
- net GND: now also C2.2, C3.2, C4.2, C5.2, R1.2, R5.1
- net GND_ESP: now also R13.2
- net GPIO3: now also SW3.2
- net GPIO4: now also R11.1; no longer SW3.2
- net GPIO5: now also R12.2, R13.1
- net VCC_2: now also C2.1, C3.1, C4.1, C5.1, R5.2, R6.1
- net VD_3.3: now also R7.1, R8.1
- net at U2.17 (~{XRSTJ}): now also R7.2
- net at BC2.2 (B): now also R11.2
- net at U2.14 (REXT): now also R1.1
- net at BC1.2 (B): now also R10.2
- net GPIO7: now reaches U1.7 (GPIO7)
- net GPIO7: now also R10.1
- net at U2.19 (BUSJ): now also R8.2
- net at U2.18 (VBUSM): now also R6.2
- net GPIO9: no longer names the net of U1.9 (GPIO9)

Commit message: update 3
Connections:
- net DATA_3_SOCKET+: now also U2.10 (DM1); no longer U2.11 (DP1)
- net DATA_3_SOCKET-: now also U2.11 (DP1); no longer U2.10 (DM1)
- net DATA_4_SOCKET+: now also U2.8 (DM2); no longer U2.9 (DP2)
- net DATA_4_SOCKET-: now also U2.9 (DP2); no longer U2.8 (DM2)
Other:
- moved on the sheet: C5, D2, J1, J4, J8, SW3, U1
