File: kicad/v1/power-control_v1.kicad_pcb (KiCad board)
At the start: 2 copper layers, 91 x 62 mm, 18 parts, among them J1 Conn_01x04_Pin, J2 USB_1, J4 Conn_01x08_Pin, J5 USB_2, J7 PINHD_2x5_Male, J8 Conn_01x02_Pin, SW1 Push_Button, SW2 Push_Button, SW3 Push_Button, U1 ESP32-C3_SUPERMINI_TH

Commit message: update 6
Parts:
- moved J1 1.54 mm to (172.6, 110.5)
Connections:
- BC2 pad 1: FP_RST_B+ -> FP_RST_B-
- SW2 pad 1: FP_RST_B- -> FP_RST_B+
- SW2 pad 2: FP_RST_B+ -> FP_RST_B-
Routing:
- net FP_RST_B-: track 45.4 -> 58.3 mm
- net FP_RST_B+: track 57.8 -> 47.9 mm
- net FP_HDD_L-: track 25.2 -> 30.1 mm
- net GPIO3: track 29.4 -> 33.7 mm
- net FP_HDD_L+: track 29.0 -> 32.5 mm
- net VCC_1: track 59.8 -> 58.0 mm
- net PSU-: track 15.5 -> 14.0 mm
- net DATA_2-: track 45.6 -> 46.5 mm
- net VCC_2: track 49.1 -> 49.9 mm
- net PSU+: track 23.6 -> 22.9 mm
- net DATA_2+: track 42.8 -> 43.4 mm
- net DATA_1+: track 29.1 -> 29.7 mm
Other:
- board text added: "GND"
- board text added: "VCC"
